File: hardware/sound-pressure-level.kicad_pcb (KiCad board)
At the start: 2 copper layers, 25 x 25 mm, 33 parts, among them P1 CON-SENSOR2, P2 BOOT, P3 DEBUG, U1 XMC1404, U2 DRILL, U3 DRILL, U4 DRILL, U5 DRILL, U6 ICS-43432, X1 16MHz

Commit message: change series resistor 220 -> 82 ohm
Parts:
- RP1: value 220 -> 82
Changed lines of the file:
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@@
-(kicad_pcb (version 4) (host pcbnew 4.0.2+dfsg1-stable)
+(kicad_pcb (version 4) (host pcbnew 4.0.7-e2-6376~58~ubuntu16.04.1)
   (general
     (links 61)
     (no_connects 0)
-    (area 129.909499 128.309499 155.290501 153.690501)
+    (area 13.96714 127.644999 155.955001 196.045)
     (thickness 1.6)
     (drawings 19)
@@
       (effects (font (size 0.2 0.2) (thickness 0.05)))
     )
-    (fp_text value 220 (at -0.025 -0.45 90) (layer F.Fab)
-      (effects (font (size 0.2 0.2) (thickness 0.05)))
-    )
+    (fp_text value 82 (at -0.025 -0.45 90) (layer F.Fab)
+      (effects (font (size 0.2 0.2) (thickness 0.05)))
+    )
